Commit message: Roughly added GQ7

File: la_z_bot_description/urdf/la_z_bot.urdf.xacro (robot description, xacro)
@@ -8,3 +8,21 @@
     <origin xyz="0.0 0.0 0.0" rpy="0 0 0"/>
   </joint>
+  <joint name="gq7_joint" type="fixed">
+    <parent link="front_mount_link" />
+    <child link="gq7_link" />
+    <origin xyz="-0.1 0.0 0.012" rpy="0 0 0"/>
+  </joint>
+  <link name="gq7_link" />
+  <joint name="gnss1_antenna_wgs84_joint" type="fixed">
+    <parent link="gq7_link" />
+    <child link="gnss1_antenna_wgs84" />
+    <origin xyz="0.0 0.5 0.0" rpy="0 0 0"/>
+  </joint>
+  <joint name="gnss2_antenna_wgs84_joint" type="fixed">
+    <parent link="gq7_link" />
+    <child link="gnss2_antenna_wgs84" />
+    <origin xyz="0.0 -0.5 0.0" rpy="0 0 0"/>
+  </joint>
+  <link name="gnss1_antenna_wgs84" />
+  <link name="gnss2_antenna_wgs84" />
 </robot>

Commit message: Bringup mostly working.  Lots of little cleanup everywhere

File: la_z_bot_description/urdf/la_z_bot.urdf.xacro (robot description, xacro)
@@ -1,15 +1,19 @@
 <?xml version="1.0"?>
-<robot name="iiwa7" xmlns:xacro="http://www.ros.org/wiki/xacro">
-  <xacro:include filename="$(find zed_wrapper)/urdf/zed_descr.urdf.xacro"/>
+<robot name="bunker" xmlns:xacro="http://www.ros.org/wiki/xacro">
   <xacro:include filename="$(find bunker_description)/urdf/bunkerPro.urdf.xacro"/>
+  <xacro:include filename="$(find zed_wrapper)/urdf/zed_macro.urdf.xacro" />
+  <xacro:zed_camera name="zed2i" model="zed2i" parent="zed_link">
+    <origin xyz="0 0 0" rpy="0 0 0" />
+  </xacro:zed_camera>
+  <link name="zed_link" />
   <joint name="zed_joint" type="fixed">
     <parent link="front_mount_link" />
     <child link="zed_link" />
-    <origin xyz="0.0 0.0 0.0" rpy="0 0 0"/>
+    <origin xyz="-0.033 0.0 0.0" rpy="0 0 0"/>
   </joint>
   <joint name="gq7_joint" type="fixed">
-    <parent link="front_mount_link" />
+    <parent link="rear_mount_link" />
     <child link="gq7_link" />
-    <origin xyz="-0.1 0.0 0.012" rpy="0 0 0"/>
+    <origin xyz="0.25 0.0 0.0" rpy="0 0 0"/>
   </joint>
   <link name="gq7_link" />
@@ -17,10 +21,10 @@
     <parent link="gq7_link" />
     <child link="gnss1_antenna_wgs84" />
-    <origin xyz="0.0 0.5 0.0" rpy="0 0 0"/>
+    <origin xyz="0.0 0.37 -0.04" rpy="0 0 0"/>
   </joint>
   <joint name="gnss2_antenna_wgs84_joint" type="fixed">
     <parent link="gq7_link" />
     <child link="gnss2_antenna_wgs84" />
-    <origin xyz="0.0 -0.5 0.0" rpy="0 0 0"/>
+    <origin xyz="0.0 -0.37 -0.04" rpy="0 0 0"/>
   </joint>
   <link name="gnss1_antenna_wgs84" />

Commit message: Added PCL and URG.  Navigation still doesn't work.  Seems like an odom issue

File: la_z_bot_description/urdf/la_z_bot.urdf.xacro (robot description, xacro)
@@ -11,4 +11,10 @@
     <child link="zed_link" />
     <origin xyz="-0.033 0.0 0.0" rpy="0 0 0"/>
+  </joint>
+  <link name="urg_link" />
+  <joint name="urg_joint" type="fixed">
+    <parent link="front_mount_link" />
+    <child link="urg_link" />
+    <origin xyz="-0.1524 0.0 0.0762" rpy="0 0 0"/>
   </joint>
   <joint name="gq7_joint" type="fixed">

Commit message: Close, but move_base is configured wrong somehow

File: la_z_bot_description/urdf/la_z_bot.urdf.xacro (robot description, xacro)
@@ -21,5 +21,5 @@
     <parent link="rear_mount_link" />
     <child link="gq7_link" />
-    <origin xyz="0.25 0.0 0.0" rpy="0 0 0"/>
+    <origin xyz="0.25 0.0 0.0" rpy="3.14159 0 0"/>
   </joint>
   <link name="gq7_link" />
@@ -27,10 +27,10 @@
     <parent link="gq7_link" />
     <child link="gnss1_antenna_wgs84" />
-    <origin xyz="0.0 0.37 -0.04" rpy="0 0 0"/>
+    <origin xyz="0.0 -0.3875 0.04" rpy="3.14159 0 0"/>
   </joint>
   <joint name="gnss2_antenna_wgs84_joint" type="fixed">
     <parent link="gq7_link" />
     <child link="gnss2_antenna_wgs84" />
-    <origin xyz="0.0 -0.37 -0.04" rpy="0 0 0"/>
+    <origin xyz="0.0 0.3875 0.04" rpy="3.14159 0 0"/>
   </joint>
   <link name="gnss1_antenna_wgs84" />

Commit message: Updated URDF for finalish component positions

File: la_z_bot_description/urdf/la_z_bot.urdf.xacro (robot description, xacro)
@@ -10,5 +10,5 @@
     <parent link="front_mount_link" />
     <child link="zed_link" />
-    <origin xyz="-0.033 0.0 0.0" rpy="0 0 0"/>
+    <origin xyz="0.0116 0.31 -0.016" rpy="3.14159 0 0"/>
   </joint>
   <link name="urg_link" />
@@ -16,10 +16,10 @@
     <parent link="front_mount_link" />
     <child link="urg_link" />
-    <origin xyz="-0.1524 0.0 0.0762" rpy="0 0 0"/>
+    <origin xyz="0 -0.32 -0.0246" rpy="3.14159 0 0"/>
   </joint>
   <joint name="gq7_joint" type="fixed">
-    <parent link="rear_mount_link" />
+    <parent link="front_mount_link" />
     <child link="gq7_link" />
-    <origin xyz="0.25 0.0 0.0" rpy="3.14159 0 0"/>
+    <origin xyz="-0.38 0.0 -0.0246" rpy="3.14159 0 0"/>
   </joint>
   <link name="gq7_link" />
@@ -27,10 +27,10 @@
     <parent link="gq7_link" />
     <child link="gnss1_antenna_wgs84" />
-    <origin xyz="0.0 -0.3875 0.04" rpy="3.14159 0 0"/>
+    <origin xyz="0.28 -0.475 0.0" rpy="3.14159 0 0"/>
   </joint>
   <joint name="gnss2_antenna_wgs84_joint" type="fixed">
     <parent link="gq7_link" />
     <child link="gnss2_antenna_wgs84" />
-    <origin xyz="0.0 0.3875 0.04" rpy="3.14159 0 0"/>
+    <origin xyz="0.28 0.475 0.0" rpy="3.14159 0 0"/>
   </joint>
   <link name="gnss1_antenna_wgs84" />

Commit message: Port of what was left on the robot

File: la_z_bot_description/urdf/la_z_bot.urdf.xacro (robot description, xacro)
@@ -21,5 +21,5 @@
     <parent link="front_mount_link" />
     <child link="gq7_link" />
-    <origin xyz="-0.38 0.0 -0.0246" rpy="3.14159 0 0"/>
+    <origin xyz="-0.36 0.0 -0.0246" rpy="3.14159 0 0"/>
   </joint>
   <link name="gq7_link" />
@@ -27,10 +27,10 @@
     <parent link="gq7_link" />
     <child link="gnss1_antenna_wgs84" />
-    <origin xyz="0.28 -0.475 0.0" rpy="3.14159 0 0"/>
+    <origin xyz="0.26 -0.475 0.0" rpy="3.14159 0 -1.5707"/>
   </joint>
   <joint name="gnss2_antenna_wgs84_joint" type="fixed">
     <parent link="gq7_link" />
     <child link="gnss2_antenna_wgs84" />
-    <origin xyz="0.28 0.475 0.0" rpy="3.14159 0 0"/>
+    <origin xyz="0.26 0.475 0.0" rpy="3.14159  0 -1.5707"/>
   </joint>
   <link name="gnss1_antenna_wgs84" />

Commit message: Added chair and side table geometry

File: la_z_bot_description/urdf/la_z_bot.urdf.xacro (robot description, xacro)
@@ -36,3 +36,16 @@
   <link name="gnss1_antenna_wgs84" />
   <link name="gnss2_antenna_wgs84" />
+  <joint name="comfy_joint" type="fixed">
+    <parent link="chassis_link" />
+    <child link="comfy_link" />
+    <origin xyz="0.0524015 0 0.460276" rpy="0 0 0"/>
+  </joint>
+  <link name="comfy_link">
+    <visual>
+      <origin xyz="0 0 0" rpy="0 0 0"/>
+      <geometry>
+        <mesh filename="package://la_z_bot_description/meshes/FrankChair.dae"/>
+      </geometry>
+    </visual>
+  </link>
 </robot>
